Commit message: Refactor robotic arm configuration and control for enhanced joint management and simulation support

File: roboticarm/src/rparm/gazebo/rparm.gazebo.xacro (robot description, xacro)
@@ -29,4 +29,5 @@
   <xacro:Link reference="${prefix}link4"/>
   <xacro:Link reference="${prefix}link5"/>
+  <xacro:Link reference="${prefix}link5_roll"/>
   <xacro:Link reference="${prefix}gripper_left_link"/>
   <xacro:Link reference="${prefix}gripper_right_link"/>
@@ -37,6 +38,9 @@
   <xacro:SimpleTransmission trans="${prefix}trans3" joint="${prefix}joint3" actuator="${prefix}actuator3" />
   <xacro:SimpleTransmission trans="${prefix}trans4" joint="${prefix}joint4" actuator="${prefix}actuator4" />
-  <xacro:SimpleTransmission trans="${prefix}trans5" joint="${prefix}gripper_left_joint" actuator="${prefix}actuator5" />
-  <xacro:SimpleTransmission trans="${prefix}trans6" joint="${prefix}gripper_right_joint" actuator="${prefix}actuator6" />
+  <xacro:SimpleTransmission trans="${prefix}trans5" joint="${prefix}joint5" actuator="${prefix}actuator5" />
+  <xacro:SimpleTransmission trans="${prefix}trans6" joint="${prefix}joint6" actuator="${prefix}actuator6" />
+  <xacro:SimpleTransmission trans="${prefix}trans7" joint="${prefix}gripper_right_joint" actuator="${prefix}actuator7" />
+  <!-- Mimic right gripper finger in sim (Harmonic / Ignition Gazebo). Keep controller at 6 joints. -->
+  <!-- No mimic plugin; control right finger directly in sim via ros2_control. -->
   </xacro:macro>
 </robot>

File: roboticarm/src/rparm/ros2_control/rparm_position.ros2_control.xacro (robot description, xacro)
@@ -14,13 +14,15 @@
           <param name="baud_rate">1000000</param>
           <param name="error_timeout_ms">500</param>
-          <param name="number_of_joints">5</param>
-          <param name="number_of_transmissions">5</param>
+          <param name="number_of_joints">6</param>
+          <param name="number_of_transmissions">6</param>
           <param name="disable_torque_at_init">true</param>
           <param name="use_revolute_to_prismatic_gripper">1</param>
-          <param name="revolute_to_prismatic_joint">${prefix}gripper_left_joint</param>
-          <param name="revolute_max">-1.52</param>
-          <param name="revolute_min">0.92</param>
-          <param name="prismatic_max">0.019</param>
-          <param name="prismatic_min">-0.01</param>
+          <!-- Map hardware gripper revolute (servo6) to URDF prismatic joint6. -->
+          <!-- Closed (neutral) ~333 deg = 5.81 rad; open target ~200 deg = 3.49 rad. -->
+          <param name="revolute_to_prismatic_joint">${prefix}joint6</param>
+          <param name="revolute_max">5.81</param>   <!-- closed/neutral -->
+          <param name="revolute_min">3.49</param>   <!-- open target -->
+          <param name="prismatic_max">0.019</param> <!-- open -->
+          <param name="prismatic_min">0.0</param>   <!-- closed/neutral -->
         </hardware>
       </xacro:unless>
@@ -49,5 +51,5 @@
         <state_interface name="effort"/>
       </joint>
-      <joint name="${prefix}gripper_left_joint">
+      <joint name="${prefix}joint5">
         <command_interface name="position"/>
         <state_interface name="position"/>
@@ -55,8 +57,14 @@
         <state_interface name="effort"/>
       </joint>
+      <joint name="${prefix}joint6">
+        <command_interface name="position"/>
+        <state_interface name="position"/>
+        <state_interface name="velocity"/>
+        <state_interface name="effort"/>
+      </joint>
+      <!-- Sim-only: expose right gripper finger to controller. -->
       <xacro:if value="$(arg use_sim)">
         <joint name="${prefix}gripper_right_joint">
-          <param name="mimic">${prefix}gripper_left_joint</param>
-          <param name="multiplier">1</param>
+          <command_interface name="position"/>
           <state_interface name="position"/>
           <state_interface name="velocity"/>

File: roboticarm/src/rparm/urdf/rparm.urdf.xacro (robot description, xacro)
@@ -17,5 +17,5 @@
     <child link="$(arg prefix)link1"/>
   </joint>
-  <xacro:rparm_arm prefix="$(arg prefix)" />
+  <xacro:rparm_arm prefix="$(arg prefix)" use_sim="$(arg use_sim)" />
   <xacro:rparm_gazebo prefix="$(arg prefix)" />
   <xacro:rparm_system

File: roboticarm/src/rparm/urdf/rparm_arm.urdf.xacro (robot description, xacro)
@@ -1,5 +1,5 @@
 <?xml version="1.0"?>
 <robot xmlns:xacro="http://www.ros.org/wiki/xacro">
-  <xacro:macro name="rparm_arm" params="prefix=''">
+  <xacro:macro name="rparm_arm" params="prefix='' use_sim:='false'">
     <xacro:property
       name="meshes_file_direction"
@@ -66,5 +66,5 @@
       <origin xyz="0.0 0.0 0.0595" rpy="0 0 0"/>
       <axis xyz="0 1 0"/>
-      <limit velocity="4.8" effort="1000" lower="${-1.5}" upper="${1.5}" />
+      <limit velocity="4.8" effort="1000" lower="${-pi}" upper="${pi}" />
       <dynamics damping="0.1"/>
     </joint>
@@ -98,5 +98,5 @@
       <origin xyz="0.024 0 0.128" rpy="0 0 0"/>
       <axis xyz="0 1 0"/>
-      <limit velocity="4.8" effort="1000" lower="${-1.5}" upper="${1.4}" />
+      <limit velocity="4.8" effort="1000" lower="${-pi}" upper="${pi}" />
       <dynamics damping="0.1"/>
     </joint>
@@ -130,5 +130,5 @@
       <origin xyz="0.124 0.0 0.0" rpy="0 0 0"/>
       <axis xyz="0 1 0"/>
-      <limit velocity="4.8" effort="1000" lower="${-1.7}" upper="${1.97}" />
+      <limit velocity="4.8" effort="1000" lower="${-pi}" upper="${pi}" />
       <dynamics damping="0.1"/>
     </joint>
@@ -157,10 +157,18 @@
       </inertial>
     </link>
-    <joint name="${prefix}gripper_left_joint" type="prismatic">
+    <!-- Wrist roll placeholder (future servo). Keep zero range so commands stay at 0. -->
+    <link name="${prefix}link5_roll">
+      <inertial>
+        <origin xyz="0 0 0" />
+        <mass value="1.0e-04" />
+        <inertia ixx="1.0e-06" ixy="0.0" ixz="0.0" iyy="1.0e-06" iyz="0.0" izz="1.0e-06" />
+      </inertial>
+    </link>
+    <joint name="${prefix}joint5" type="revolute">
       <parent link="${prefix}link5"/>
-      <child link="${prefix}gripper_left_link"/>
-      <origin xyz="0.0817 0.021 0.0" rpy="0 0 0"/>
-      <axis xyz="0 1 0"/>
-      <limit velocity="4.8" effort="1000" lower="-0.011" upper="0.02" />
+      <child link="${prefix}link5_roll"/>
+      <origin xyz="0 0 0" rpy="0 0 0"/>
+      <axis xyz="0 0 1"/>
+      <limit velocity="4.8" effort="1000" lower="0" upper="0" />
       <dynamics damping="0.1"/>
     </joint>
@@ -189,13 +197,35 @@
       </inertial>
     </link>
-    <joint name="${prefix}gripper_right_joint" type="prismatic">
-      <parent link="${prefix}link5"/>
-      <child link="${prefix}gripper_right_link"/>
-      <origin xyz="0.0817 -0.021 0" rpy="0 0 0"/>
-      <axis xyz="0 -1 0"/>
+    <joint name="${prefix}joint6" type="prismatic">
+      <parent link="${prefix}link5_roll"/>
+      <child link="${prefix}gripper_left_link"/>
+      <origin xyz="0.0817 0.021 0.0" rpy="0 0 0"/>
+      <axis xyz="0 1 0"/>
       <limit velocity="4.8" effort="1000" lower="-0.011" upper="0.02" />
-      <dynamics damping="0.7"/>
-      <mimic joint="${prefix}gripper_left_joint" multiplier="1"/>
-    </joint>
+      <dynamics damping="0.1"/>
+    </joint>
+    <xacro:if value="${use_sim}">
+      <!-- Sim: control right finger independently (no mimic) so ros2_control can drive both. -->
+      <joint name="${prefix}gripper_right_joint" type="prismatic">
+        <parent link="${prefix}link5_roll"/>
+        <child link="${prefix}gripper_right_link"/>
+        <origin xyz="0.0817 -0.021 0" rpy="0 0 0"/>
+        <axis xyz="0 -1 0"/>
+        <limit velocity="4.8" effort="1000" lower="-0.011" upper="0.02" />
+        <dynamics damping="0.7"/>
+      </joint>
+    </xacro:if>
+    <xacro:unless value="${use_sim}">
+      <!-- Hardware: keep mimic description (handled in bridge) -->
+      <joint name="${prefix}gripper_right_joint" type="prismatic">
+        <parent link="${prefix}link5_roll"/>
+        <child link="${prefix}gripper_right_link"/>
+        <origin xyz="0.0817 -0.021 0" rpy="0 0 0"/>
+        <axis xyz="0 -1 0"/>
+        <limit velocity="4.8" effort="1000" lower="-0.011" upper="0.02" />
+        <dynamics damping="0.7"/>
+        <mimic joint="${prefix}joint6" multiplier="1"/>
+      </joint>
+    </xacro:unless>
     <link name="${prefix}gripper_right_link">
       <visual>
